Commit message: A1: used descriptive variable names

File: urdf/agv.gazebo.xacro (robot description, xacro)
@@ -3,6 +3,7 @@
   <xacro:arg name="laser_visual" default="true"/>
   <xacro:arg name="imu_visual"   default="true"/>
+  <!-- Differential Drive Controller Plugin -->
   <gazebo>
-    <plugin name="turtlebot3_burger_controller" filename="libgazebo_ros_diff_drive.so">
+    <plugin name="differential_drive_controller" filename="libgazebo_ros_diff_drive.so">
       <commandTopic>cmd_vel</commandTopic>
       <rosDebugLevel>Debug</rosDebugLevel>
@@ -26,4 +27,5 @@
     <material>Gazebo/Grey</material>
   </gazebo>
+  <!-- Drive Wheel Properties -->
   <gazebo reference="left_wheel_joint">
     <mu1>1000000.0</mu1>
@@ -46,5 +48,6 @@
     <material>Gazebo/Grey</material>
   </gazebo>
-  <gazebo reference="caster_left_back_joint">
+  <!-- Caster Wheel Joint Properties -->
+  <gazebo reference="left_caster_back_joint">
     <mu1>1.0</mu1>
     <mu2>0.0</mu2>
@@ -55,5 +58,5 @@
     <material>Gazebo/Grey</material>
   </gazebo>
-  <gazebo reference="caster_right_back_joint">
+  <gazebo reference="right_caster_back_joint">
     <mu1>1.0</mu1>
     <mu2>0.0</mu2>
@@ -64,5 +67,5 @@
     <material>Gazebo/Grey</material>
   </gazebo>
-  <gazebo reference="caster_left_front_joint">
+  <gazebo reference="left_caster_front_joint">
     <mu1>1.0</mu1>
     <mu2>0.0</mu2>
@@ -73,5 +76,5 @@
     <material>Gazebo/Grey</material>
   </gazebo>
-  <gazebo reference="caster_right_front_joint">
+  <gazebo reference="right_caster_front_joint">
     <mu1>1.0</mu1>
     <mu2>0.0</mu2>
@@ -82,6 +85,7 @@
     <material>Gazebo/Grey</material>
   </gazebo>
+  <!-- IMU Sensor Plugin -->
   <gazebo>
-    <plugin name="imu_plugin" filename="libgazebo_ros_imu.so">
+    <plugin name="imu_sensor_plugin" filename="libgazebo_ros_imu.so">
       <alwaysOn>true</alwaysOn>
       <bodyName>imu_link</bodyName>
@@ -110,5 +114,5 @@
   </gazebo>
   <gazebo reference="imu_link">
-    <sensor type="imu" name="imu">
+    <sensor type="imu" name="imu_sensor">
       <always_on>true</always_on>
       <update_rate>100</update_rate>
@@ -117,7 +121,8 @@
     <material>Gazebo/Grey</material>
   </gazebo>
-  <gazebo reference="base_scan">
+  <!-- Front Laser Scanner Sensor -->
+  <gazebo reference="laser_front_link">
     <material>Gazebo/Blue</material>
-    <sensor type="ray" name="lds_lfcd_sensor">
+    <sensor type="ray" name="front_laser_sensor">
       <pose>0.0 0.0 0.0 0 0 0</pose>
       <visualize>$(arg laser_visual)</visualize>
@@ -143,7 +148,7 @@
         </noise>
       </ray>
-      <plugin name="gazebo_ros_lds_lfcd_controller" filename="libgazebo_ros_laser.so">
-        <topicName>scan///</topicName>
-        <frameName>base_scan</frameName>
+      <plugin name="front_laser_controller" filename="libgazebo_ros_laser.so">
+        <topicName>scan</topicName>
+        <frameName>laser_front_link</frameName>
       </plugin>
     </sensor>

File: urdf/agv.macros.xacro (robot description, xacro)
@@ -1,129 +1,133 @@
 <?xml version="1.0"?>
 <robot xmlns:xacro="http://ros.org/wiki/xacro">
-     <xacro:macro name="cylinder_inertia" params="m r h">
-        <inertia  ixx="${m*(3*r*r+h*h)/12}" ixy = "0" ixz = "0"
-                  iyy="${m*(3*r*r+h*h)/12}" iyz = "0"
-                  izz="${m*r*r/2}" />
-      </xacro:macro>
-      <xacro:macro name="box_inertia" params="m x y z">
-        <inertia  ixx="${m*(y*y+z*z)/12}" ixy = "0" ixz = "0"
-                  iyy="${m*(x*x+z*z)/12}" iyz = "0"
-                  izz="${m*(x*x+z*z)/12}" />
-      </xacro:macro>
-      <xacro:macro name="sphere_inertia" params="m r">
-        <inertia  ixx="${2*m*r*r/5}" ixy = "0" ixz = "0"
-                  iyy="${2*m*r*r/5}" iyz = "0"
-                  izz="${2*m*r*r/5}" />
- </xacro:macro>
- <xacro:macro name="wheel" params="lr tY">
-     <joint name="${lr}_wheel_joint" type="continuous">
-        <parent link="base_link"/>
-        <child link="${lr}_wheel"/>
-        <origin xyz="0.0 ${tY} -0.04625" rpy="-1.57 0 0"/>
-        <axis xyz="0 0 1"/>
-      </joint>
-      <link name="${lr}_wheel">
-        <visual>
-          <origin xyz="0 0 0" rpy="0 0 0"/>
-          <geometry>
-           <cylinder length="${wheelWidth}" radius="${wheelRadius}"/>
-          </geometry>
-          <material name="black"/>
-        </visual>
-        <collision>
-            <origin xyz="0 0 0" rpy="0 0 0" />
-          <geometry>
-          <cylinder length="${wheelWidth}" radius="${wheelRadius}"/>
-          </geometry>
-        </collision>
-        <inertial>
-      	 <origin xyz="0 0 0" />
-      	 <mass value="2.6" />
-      	 <inertia ixx="0.01300" ixy="0.0" ixz="0.0"
-               iyy="0.007042" iyz="0.0"
-               izz="0.007042" />
-    	</inertial>
-        <gazebo reference="${lr}_wheel">
-	     <mu1>10.0</mu1>
-	     <mu2>10.0</mu2>
-	     <kp>500000.0</kp>
-	     <kd>10.0</kd>
-	     <maxVel>1.1</maxVel>
-	     <material>Gazebo/Black</material>
-        </gazebo>
-	  </link>
-    </xacro:macro>
-<xacro:macro name="caster_front" params="lr tY">
-       <joint name="${lr}_caster_front_joint" type="fixed">
-        <parent link="base_link"/>
-        <child link="${lr}_caster_front"/>
-        <origin xyz="0.650 ${tY} -0.109" rpy="0 0 0"/>
-       </joint>
-       <link name="${lr}_caster_front">
-        <visual>
-          <origin xyz="0 0 0" rpy="0 ${M_PI/2} 0" />
-          <geometry>
-           <sphere radius="${casterRadius}" />
-          </geometry>
-          <material name="blue"/>
-        </visual>
-        <collision>
-            <origin xyz="0 0 0" rpy="0 ${M_PI/2} 0" />
-          <geometry>
-           <sphere radius="${casterRadius}"/>
-          </geometry>
-        </collision>
-        <inertial>
-          <origin xyz="0 0 0" rpy="0 ${M_PI/2} 0" />
-          <mass value="${casterMass}"/>
-          <sphere_inertia m="${casterMass}" r="${casterRadius}"/>
-        </inertial>
-       </link>
-       <gazebo reference="${lr}_caster_front">
-	     <mu1>0.0</mu1>
-	     <mu2>0.0</mu2>
-	     <kp>1000000.0</kp>
-	     <kd>100.0</kd>
-	     <maxVel>1.0</maxVel>
-	     <material>Gazebo/Blue</material>
-       </gazebo>
- </xacro:macro>
- <xacro:macro name="caster_back" params="lr tY">
-     <joint name="${lr}_caster_back_joint" type="fixed">
-        <parent link="base_link"/>
-        <child link="${lr}_caster_back"/>
-        <origin xyz="-0.650 ${tY} -0.109" rpy="0 0 0"/>
-	    <axis xyz="0 0 1"/>
-      </joint>
-      <link name="${lr}_caster_back">
-        <visual>
-          <origin xyz="0 0 0" rpy="0 ${M_PI/2} 0" />
-          <geometry>
-           <sphere radius="${casterRadius}" />
-          </geometry>
-          <material name="blue"/>
-        </visual>
-        <collision>
-            <origin xyz="0 0 0" rpy="0 ${M_PI/2} 0" />
-          <geometry>
-           <sphere radius="${casterRadius}" />
-          </geometry>
-        </collision>
-        <inertial>
-       		<origin xyz="0 0 0.0" />
-      		<mass value="0.01" />
-      		<inertia ixx="0.001" ixy="0.0" ixz="0.0"
-       	        	iyy="0.001" iyz="0.0"
-               		izz="0.0001" />
-       </inertial>
-      </link>
-      <gazebo reference="${lr}_caster_back">
-	    <mu1>1.0</mu1>
-	    <mu2>1.0</mu2>
-	    <kp>1000000.0</kp>
-	    <kd>10.0</kd>
-	    <maxVel>3.0</maxVel>
-	    <material>Gazebo/Blue</material>
+  <!-- Inertia Calculation Macros -->
+  <xacro:macro name="cylinder_inertia" params="mass radius length">
+    <inertia  ixx="${mass*(3*radius*radius + length*length)/12}" ixy="0" ixz="0"
+              iyy="${mass*(3*radius*radius + length*length)/12}" iyz="0"
+              izz="${mass*radius*radius/2}" />
+  </xacro:macro>
+  <xacro:macro name="box_inertia" params="mass size_x size_y size_z">
+    <inertia  ixx="${mass*(size_y*size_y + size_z*size_z)/12}" ixy="0" ixz="0"
+              iyy="${mass*(size_x*size_x + size_z*size_z)/12}" iyz="0"
+              izz="${mass*(size_x*size_x + size_z*size_z)/12}" />
+  </xacro:macro>
+  <xacro:macro name="sphere_inertia" params="mass radius">
+    <inertia  ixx="${2*mass*radius*radius/5}" ixy="0" ixz="0"
+              iyy="${2*mass*radius*radius/5}" iyz="0"
+              izz="${2*mass*radius*radius/5}" />
+  </xacro:macro>
+  <!-- Drive Wheel Macro -->
+  <xacro:macro name="wheel" params="wheel_side offset_y">
+    <joint name="${wheel_side}_wheel_joint" type="continuous">
+      <parent link="base_link"/>
+      <child link="${wheel_side}_wheel"/>
+      <origin xyz="0.0 ${offset_y} -0.04625" rpy="-1.57 0 0"/>
+      <axis xyz="0 0 1"/>
+    </joint>
+    <link name="${wheel_side}_wheel">
+      <visual>
+        <origin xyz="0 0 0" rpy="0 0 0"/>
+        <geometry>
+          <cylinder length="${wheel_width}" radius="${wheel_radius}"/>
+        </geometry>
+        <material name="black"/>
+      </visual>
+      <collision>
+        <origin xyz="0 0 0" rpy="0 0 0" />
+        <geometry>
+          <cylinder length="${wheel_width}" radius="${wheel_radius}"/>
+        </geometry>
+      </collision>
+      <inertial>
+        <origin xyz="0 0 0" />
+        <mass value="${wheel_mass}" />
+        <inertia ixx="0.01300" ixy="0.0" ixz="0.0"
+                 iyy="0.007042" iyz="0.0"
+                 izz="0.007042" />
+      </inertial>
+      <gazebo reference="${wheel_side}_wheel">
+        <mu1>10.0</mu1>
+        <mu2>10.0</mu2>
+        <kp>500000.0</kp>
+        <kd>10.0</kd>
+        <maxVel>1.1</maxVel>
+        <material>Gazebo/Black</material>
       </gazebo>
+    </link>
+  </xacro:macro>
+  <!-- Front Caster Wheel Macro -->
+  <xacro:macro name="caster_front" params="caster_side offset_y">
+    <joint name="${caster_side}_caster_front_joint" type="fixed">
+      <parent link="base_link"/>
+      <child link="${caster_side}_caster_front"/>
+      <origin xyz="0.650 ${offset_y} -0.109" rpy="0 0 0"/>
+    </joint>
+    <link name="${caster_side}_caster_front">
+      <visual>
+        <origin xyz="0 0 0" rpy="0 ${M_PI/2} 0" />
+        <geometry>
+          <sphere radius="${caster_radius}" />
+        </geometry>
+        <material name="blue"/>
+      </visual>
+      <collision>
+        <origin xyz="0 0 0" rpy="0 ${M_PI/2} 0" />
+        <geometry>
+          <sphere radius="${caster_radius}"/>
+        </geometry>
+      </collision>
+      <inertial>
+        <origin xyz="0 0 0" rpy="0 ${M_PI/2} 0" />
+        <mass value="${caster_mass}"/>
+        <sphere_inertia mass="${caster_mass}" radius="${caster_radius}"/>
+      </inertial>
+    </link>
+    <gazebo reference="${caster_side}_caster_front">
+      <mu1>0.0</mu1>
+      <mu2>0.0</mu2>
+      <kp>1000000.0</kp>
+      <kd>100.0</kd>
+      <maxVel>1.0</maxVel>
+      <material>Gazebo/Blue</material>
+    </gazebo>
+  </xacro:macro>
+  <!-- Back Caster Wheel Macro -->
+  <xacro:macro name="caster_back" params="caster_side offset_y">
+    <joint name="${caster_side}_caster_back_joint" type="fixed">
+      <parent link="base_link"/>
+      <child link="${caster_side}_caster_back"/>
+      <origin xyz="-0.650 ${offset_y} -0.109" rpy="0 0 0"/>
+      <axis xyz="0 0 1"/>
+    </joint>
+    <link name="${caster_side}_caster_back">
+      <visual>
+        <origin xyz="0 0 0" rpy="0 ${M_PI/2} 0" />
+        <geometry>
+          <sphere radius="${caster_radius}" />
+        </geometry>
+        <material name="blue"/>
+      </visual>
+      <collision>
+        <origin xyz="0 0 0" rpy="0 ${M_PI/2} 0" />
+        <geometry>
+          <sphere radius="${caster_radius}" />
+        </geometry>
+      </collision>
+      <inertial>
+        <origin xyz="0 0 0.0" />
+        <mass value="0.01" />
+        <inertia ixx="0.001" ixy="0.0" ixz="0.0"
+                 iyy="0.001" iyz="0.0"
+                 izz="0.0001" />
+      </inertial>
+    </link>
+    <gazebo reference="${caster_side}_caster_back">
+      <mu1>1.0</mu1>
+      <mu2>1.0</mu2>
+      <kp>1000000.0</kp>
+      <kd>10.0</kd>
+      <maxVel>3.0</maxVel>
+      <material>Gazebo/Blue</material>
+    </gazebo>
   </xacro:macro>
 </robot>

File: urdf/agv.urdf.xacro (robot description, xacro)
@@ -1,19 +1,25 @@
 <?xml version="1.0" ?>
 <robot name="agv" xmlns:xacro="http://ros.org/wiki/xacro">
+  <!-- General Arguments & Constants -->
   <xacro:arg name="robot_namespace" default="/" />
   <xacro:property name="M_PI" value="3.1415926535897931"/>
-  <xacro:property name="chassisLength" value="1.558"/>
-  <xacro:property name="chassisWidth" value="0.965"/>
-  <xacro:property name="chassisHeight" value="0.280"/>
-  <xacro:property name="chassisMass" value="300"/>
-  <xacro:property name="casterRadius" value="0.062"/>
-  <xacro:property name="casterLength" value="0.05"/>
-  <xacro:property name="casterMass" value="5.2"/>
-  <xacro:property name="wheelWidth" value="0.05"/>
-  <xacro:property name="wheelRadius" value="0.1"/>
-  <xacro:property name="wheelMass" value="2"/>
+  <!-- Chassis Physical Dimensions & Mass -->
+  <xacro:property name="chassis_length" value="1.558"/>
+  <xacro:property name="chassis_width" value="0.965"/>
+  <xacro:property name="chassis_height" value="0.280"/>
+  <xacro:property name="chassis_mass" value="300"/>
+  <!-- Caster Wheel Physical Dimensions & Mass -->
+  <xacro:property name="caster_radius" value="0.062"/>
+  <xacro:property name="caster_length" value="0.05"/>
+  <xacro:property name="caster_mass" value="5.2"/>
+  <!-- Drive Wheel Physical Dimensions & Mass -->
+  <xacro:property name="wheel_width" value="0.05"/>
+  <xacro:property name="wheel_radius" value="0.1"/>
+  <xacro:property name="wheel_mass" value="2"/>
+  <!-- Path and Model Arguments -->
   <xacro:arg name="config_path" default="" />
   <xacro:arg name="robot_model" default="$(env AMR_MODEL)"/>
   <xacro:arg name="parameters_dir" default="$(env ROS_PACKAGE_PATH)"/>
+  <!-- Included Xacro Files -->
   <xacro:include filename="$(arg parameters_dir)/Product/$(arg robot_model)/RobotUrdf/common_properties.xacro"/>
   <xacro:include filename="$(arg config_path)/_CONFIG_/laser_correction.xacro"/>
@@ -22,21 +28,23 @@
   <xacro:include filename="$(arg parameters_dir)/Product/$(arg robot_model)/RobotUrdf/agv.gazebo.xacro"/>
   <xacro:include filename="$(arg parameters_dir)/Product/$(arg robot_model)/RobotUrdf/agv.macros.xacro"/>
+  <!-- Base Footprint (Ground Projection Link) -->
   <link name="base_footprint"/>
-  <joint name="base_joint" type="fixed">
+  <joint name="base_footprint_to_base_link_joint" type="fixed">
     <parent link="base_footprint"/>
     <child link="base_link"/>
     <origin xyz="0.0 0.0 0.0" rpy="0 0 0"/>
   </joint>
+  <!-- Chassis Base Link -->
   <link name="base_link">
     <collision>
-      <origin xyz="0 0 0" rpy="0 0  0"/>
-      <geometry>
-	<box size="${chassisLength} ${chassisWidth} ${chassisHeight}"/>
-      </geometry>
-    </collision>
-    <visual>
       <origin xyz="0 0 0" rpy="0 0 0"/>
       <geometry>
-	<box size="${chassisLength} ${chassisWidth} ${chassisHeight}"/>
+        <box size="${chassis_length} ${chassis_width} ${chassis_height}"/>
+      </geometry>
+    </collision>
+    <visual>
+      <origin xyz="0 0 0" rpy="0 0 0"/>
+      <geometry>
+        <box size="${chassis_length} ${chassis_width} ${chassis_height}"/>
       </geometry>
       <material name="grey"/>
@@ -44,5 +52,5 @@
     <inertial>
       <origin xyz="0 0 0" />
-      <mass value="${chassisMass}" />
+      <mass value="${chassis_mass}" />
       <inertia ixx="3.9687"
         ixy="0.28534"
@@ -52,12 +60,15 @@
         izz="8.1939" />
     </inertial>
-   </link>
-  <wheel lr="left" tY="0.40649"/>
-  <wheel lr="right" tY="-0.40649"/>
-  <caster_front lr="left" tY="0.400"/>
-  <caster_front lr="right" tY="-0.400"/>
-  <caster_back lr="left" tY="0.400" />
-  <caster_back lr="right" tY="-0.400"/>
-  <link name="laser1">
+  </link>
+  <!-- Drive Wheels -->
+  <wheel wheel_side="left" offset_y="0.40649"/>
+  <wheel wheel_side="right" offset_y="-0.40649"/>
+  <!-- Caster Wheels (Front & Back) -->
+  <caster_front caster_side="left" offset_y="0.400"/>
+  <caster_front caster_side="right" offset_y="-0.400"/>
+  <caster_back caster_side="left" offset_y="0.400" />
+  <caster_back caster_side="right" offset_y="-0.400"/>
+  <!-- Front Laser Scanner -->
+  <link name="laser_front_link">
     <visual>
       <origin xyz="0.0 0.0 0.0" rpy="0 0 0"/>
@@ -84,5 +95,11 @@
     </inertial>
   </link>
-  <link name="laser2">
+  <joint name="laser_front_joint" type="fixed">
+    <parent link="base_link"/>
+    <child link="laser_front_link"/>
+    <origin xyz="${laser_front_x} ${laser_front_y} ${laser_front_z}" rpy="${laser_front_roll} ${laser_front_pitch} ${laser_front_yaw}"/>
+  </joint>
+  <!-- Back Laser Scanner -->
+  <link name="laser_back_link">
     <visual>
       <origin xyz="0.0 0.0 0.0" rpy="0 0 0"/>
@@ -101,5 +118,5 @@
       <mass value="0.5925" />
       <origin xyz="-7.8839E-05 4.3846E-05 -0.016941" rpy="0 0 0" />
-      <inertia  ixx="0.00070857"
+      <inertia ixx="0.00070857"
         ixy="-1.3137E-06"
         ixz="1.6001E-06"
@@ -109,20 +126,11 @@
     </inertial>
   </link>
-  <joint name="scan_joint_back" type="fixed">
-    <parent link="base_link"/>
-    <child link="laser2"/>
+  <joint name="laser_back_joint" type="fixed">
+    <parent link="base_link"/>
+    <child link="laser_back_link"/>
     <origin xyz="${laser_back_x} ${laser_back_y} ${laser_back_z}" rpy="${laser_back_roll} ${laser_back_pitch} ${laser_back_yaw}"/>
   </joint>
-  <joint name="scan_joint_front" type="fixed">
-    <parent link="base_link"/>
-    <child link="laser1"/>
-    <origin xyz="${laser_front_x} ${laser_front_y} ${laser_front_z}" rpy="${laser_front_roll} ${laser_front_pitch} ${laser_front_yaw}"/>
-  </joint>
-  <joint name="scan_3d" type="fixed">
-    <parent link="base_link"/>
-    <child link="laser_3d"/>
-    <origin xyz="${laser_3d_x} ${laser_3d_y} ${laser_3d_z}" rpy="${laser_3d_roll} ${laser_3d_pitch} ${laser_3d_yaw}"/>
-  </joint>
-  <link name="laser_3d">
+  <!-- 3D Laser Scanner -->
+  <link name="laser_3d_link">
     <visual>
       <origin xyz="0.0 0.0 0.0" rpy="0 0 0"/>
@@ -146,10 +154,18 @@
     </inertial>
   </link>
-  <link name="laser"/>
-  <joint name="scan_pnf" type="fixed">
-    <parent link="base_link"/>
-    <child link="laser"/>
+  <joint name="laser_3d_joint" type="fixed">
+    <parent link="base_link"/>
+    <child link="laser_3d_link"/>
+    <origin xyz="${laser_3d_x} ${laser_3d_y} ${laser_3d_z}" rpy="${laser_3d_roll} ${laser_3d_pitch} ${laser_3d_yaw}"/>
+  </joint>
+  <!-- Primary / PNF Laser Link -->
+  <link name="laser_pnf_link"/>
+  <joint name="laser_pnf_joint" type="fixed">
+    <parent link="base_link"/>
+    <child link="laser_pnf_link"/>
     <origin xyz="${laser_x} ${laser_y} ${laser_z}" rpy="${laser_roll} ${laser_pitch} ${laser_yaw}"/>
   </joint>
+  <!-- IMU Sensor -->
+  <link name="imu_link"/>
   <joint name="imu_joint" type="fixed">
     <parent link="base_link"/>
@@ -157,62 +173,41 @@
     <origin xyz="${imu_x} ${imu_y} ${imu_z}" rpy="${imu_roll} ${imu_pitch} ${imu_yaw}"/>
   </joint>
-  <link name="imu_link"/>
-  <link name="camera1_link"/>
-  <joint name="camera1joint" type="fixed">
-    <!--origin
-      xyz="0.73448 0.1567 0.1225"
-	    rpy="0 0 -0.5236" /-->
-    <origin xyz="${camera1_x} ${camera1_y} ${camera1_z}" rpy="${camera1_roll} ${camera1_pitch} ${camera1_yaw}"/>
-    <parent
-      link="base_link" />
-    <child
-      link="camera1_link" />
-    <axis
-      xyz="0 0 0" />
-  </joint>
-<link name="camera1_color_optical_frame"/>
-  <joint name="optical_joint1" type="fixed">
-    <parent link="camera1_link"/>
-    <child link="camera1_color_optical_frame"/>
+  <!-- Camera 1 -->
+  <link name="camera_1_link"/>
+  <joint name="camera_1_joint" type="fixed">
+    <origin xyz="${camera_1_x} ${camera_1_y} ${camera_1_z}" rpy="${camera_1_roll} ${camera_1_pitch} ${camera_1_yaw}"/>
+    <parent link="base_link"/>
+    <child link="camera_1_link"/>
+    <axis xyz="0 0 0"/>
+  </joint>
+  <link name="camera_1_color_optical_frame"/>
+  <joint name="camera_1_color_optical_joint" type="fixed">
+    <parent link="camera_1_link"/>
+    <child link="camera_1_color_optical_frame"/>
     <origin xyz="0.0 0.0 0.0" rpy="-1.57 0.0 -1.57"/>
   </joint>
-   <link name="camera2_link"/>
-  <joint name="camera2joint" type="fixed">
-    <!--origin
-      xyz="0.73448 -0.1567 0.1225"
-	    rpy="0 0 0.5236" /-->
-    <origin xyz="${camera2_x} ${camera2_y} ${camera2_z}" rpy="${camera2_roll} ${camera2_pitch} ${camera2_yaw}"/>
-    <parent
-      link="base_link" />
-    <child
-      link="camera2_link" />
-    <axis
-      xyz="0 0 0" />
-  </joint>
-  <link name="camera3_link"/>
-  <joint name="camera3joint" type="fixed">
-    <!--origin
-      xyz="-0.73558 -0.1568 0.1225"
-      rpy="0 0 2.618" /-->
-    <origin xyz="${camera3_x} ${camera3_y} ${camera3_z}" rpy="${camera3_roll} ${camera3_pitch} ${camera3_yaw}"/>
-    <parent
-      link="base_link" />
-    <child
-      link="camera3_link" />
-    <axis
-      xyz="0 0 0" />
-  </joint>
-  <link name="camera4_link"/>
-  <joint name="camera4joint" type="fixed">
-    <!--origin
-      xyz="-0.73558 0.1568 0.1225"
-      rpy="0 0 -2.618" /-->
-    <origin xyz="${camera4_x} ${camera4_y} ${camera4_z}" rpy="${camera4_roll} ${camera4_pitch} ${camera4_yaw}"/>
-    <parent
-      link="base_link" />
-    <child
-      link="camera4_link" />
-    <axis
-      xyz="0 0 0" />
+  <!-- Camera 2 -->
+  <link name="camera_2_link"/>
+  <joint name="camera_2_joint" type="fixed">
+    <origin xyz="${camera_2_x} ${camera_2_y} ${camera_2_z}" rpy="${camera_2_roll} ${camera_2_pitch} ${camera_2_yaw}"/>
+    <parent link="base_link"/>
+    <child link="camera_2_link"/>
+    <axis xyz="0 0 0"/>
+  </joint>
+  <!-- Camera 3 -->
+  <link name="camera_3_link"/>
+  <joint name="camera_3_joint" type="fixed">
+    <origin xyz="${camera_3_x} ${camera_3_y} ${camera_3_z}" rpy="${camera_3_roll} ${camera_3_pitch} ${camera_3_yaw}"/>
+    <parent link="base_link"/>
+    <child link="camera_3_link"/>
+    <axis xyz="0 0 0"/>
+  </joint>
+  <!-- Camera 4 -->
+  <link name="camera_4_link"/>
+  <joint name="camera_4_joint" type="fixed">
+    <origin xyz="${camera_4_x} ${camera_4_y} ${camera_4_z}" rpy="${camera_4_roll} ${camera_4_pitch} ${camera_4_yaw}"/>
+    <parent link="base_link"/>
+    <child link="camera_4_link"/>
+    <axis xyz="0 0 0"/>
   </joint>
 </robot>
