Commit message: A2: modified urd files for modularity

File: urdf/agv.gazebo.xacro (robot description, xacro)
@@ -18,5 +18,5 @@
       <leftJoint>left_wheel_joint</leftJoint>
       <rightJoint>right_wheel_joint</rightJoint>
-      <wheelSeparation>0.654</wheelSeparation>
+      <wheelSeparation>0.81298</wheelSeparation>
       <wheelDiameter>0.200</wheelDiameter>
       <wheelAcceleration>1</wheelAcceleration>
@@ -27,6 +27,6 @@
     <material>Gazebo/Grey</material>
   </gazebo>
-  <!-- Drive Wheel Properties -->
-  <gazebo reference="left_wheel_joint">
+  <!-- Drive Wheel Contact Properties -->
+  <gazebo reference="left_wheel">
     <mu1>1000000.0</mu1>
     <mu2>100000.0</mu2>
@@ -38,5 +38,5 @@
     <material>Gazebo/Grey</material>
   </gazebo>
-  <gazebo reference="right_wheel_joint">
+  <gazebo reference="right_wheel">
     <mu1>1000000.0</mu1>
     <mu2>100000.0</mu2>
@@ -46,41 +46,4 @@
     <maxVel>0.8</maxVel>
     <fdir1>1 0 0</fdir1>
-    <material>Gazebo/Grey</material>
-  </gazebo>
-  <!-- Caster Wheel Joint Properties -->
-  <gazebo reference="left_caster_back_joint">
-    <mu1>1.0</mu1>
-    <mu2>0.0</mu2>
-    <kp>1000000.0</kp>
-    <kd>100.0</kd>
-    <minDepth>0.01</minDepth>
-    <maxVel>1.0</maxVel>
-    <material>Gazebo/Grey</material>
-  </gazebo>
-  <gazebo reference="right_caster_back_joint">
-    <mu1>1.0</mu1>
-    <mu2>0.0</mu2>
-    <kp>1000000.0</kp>
-    <kd>100.0</kd>
-    <minDepth>0.01</minDepth>
-    <maxVel>1.0</maxVel>
-    <material>Gazebo/Grey</material>
-  </gazebo>
-  <gazebo reference="left_caster_front_joint">
-    <mu1>1.0</mu1>
-    <mu2>0.0</mu2>
-    <kp>1000000.0</kp>
-    <kd>100.0</kd>
-    <minDepth>0.01</minDepth>
-    <maxVel>1.0</maxVel>
-    <material>Gazebo/Grey</material>
-  </gazebo>
-  <gazebo reference="right_caster_front_joint">
-    <mu1>1.0</mu1>
-    <mu2>0.0</mu2>
-    <kp>1000000.0</kp>
-    <kd>100.0</kd>
-    <minDepth>0.01</minDepth>
-    <maxVel>1.0</maxVel>
     <material>Gazebo/Grey</material>
   </gazebo>
@@ -121,36 +84,41 @@
     <material>Gazebo/Grey</material>
   </gazebo>
-  <!-- Front Laser Scanner Sensor -->
-  <gazebo reference="laser_front_link">
-    <material>Gazebo/Blue</material>
-    <sensor type="ray" name="front_laser_sensor">
-      <pose>0.0 0.0 0.0 0 0 0</pose>
-      <visualize>$(arg laser_visual)</visualize>
-      <update_rate>18.0</update_rate>
-      <ray>
-        <scan>
-          <horizontal>
-            <samples>360</samples>
-            <resolution>1</resolution>
-            <min_angle>-0.67</min_angle>
-            <max_angle>3.84</max_angle>
-          </horizontal>
-        </scan>
-        <range>
-          <min>0.120</min>
-          <max>8.5</max>
-          <resolution>0.025</resolution>
-        </range>
-        <noise>
-          <type>gaussian</type>
-          <mean>0.0</mean>
-          <stddev>0.01</stddev>
-        </noise>
-      </ray>
-      <plugin name="front_laser_controller" filename="libgazebo_ros_laser.so">
-        <topicName>scan</topicName>
-        <frameName>laser_front_link</frameName>
-      </plugin>
-    </sensor>
-  </gazebo>
+  <!-- Laser Sensor Plugin Macro -->
+  <xacro:macro name="gazebo_laser_plugin" params="link_name sensor_name topic_name update_rate:=18.0 min_angle:=-3.14159 max_angle:=3.14159">
+    <gazebo reference="${link_name}">
+      <material>Gazebo/Blue</material>
+      <sensor type="ray" name="${sensor_name}">
+        <pose>0 0 0 0 0 0</pose>
+        <visualize>$(arg laser_visual)</visualize>
+        <update_rate>${update_rate}</update_rate>
+        <ray>
+          <scan>
+            <horizontal>
+              <samples>360</samples>
+              <resolution>1</resolution>
+              <min_angle>${min_angle}</min_angle>
+              <max_angle>${max_angle}</max_angle>
+            </horizontal>
+          </scan>
+          <range>
+            <min>0.120</min>
+            <max>10.0</max>
+            <resolution>0.025</resolution>
+          </range>
+          <noise>
+            <type>gaussian</type>
+            <mean>0.0</mean>
+            <stddev>0.01</stddev>
+          </noise>
+        </ray>
+        <plugin name="${sensor_name}_controller" filename="libgazebo_ros_laser.so">
+          <topicName>${topic_name}</topicName>
+          <frameName>${link_name}</frameName>
+        </plugin>
+      </sensor>
+    </gazebo>
+  </xacro:macro>
+  <!-- Front and Back 2D Laser Ray Sensors -->
+  <xacro:gazebo_laser_plugin link_name="laser_front_link" sensor_name="front_laser" topic_name="scan_front"/>
+  <xacro:gazebo_laser_plugin link_name="laser_back_link"  sensor_name="back_laser"  topic_name="scan_back"/>
 </robot>

File: urdf/agv.macros.xacro (robot description, xacro)
@@ -1,5 +1,5 @@
 <?xml version="1.0"?>
 <robot xmlns:xacro="http://ros.org/wiki/xacro">
-  <!-- Inertia Calculation Macros -->
+  <!-- Inertia Calculation Helpers -->
   <xacro:macro name="cylinder_inertia" params="mass radius length">
     <inertia  ixx="${mass*(3*radius*radius + length*length)/12}" ixy="0" ixz="0"
@@ -13,7 +13,7 @@
   </xacro:macro>
   <xacro:macro name="sphere_inertia" params="mass radius">
-    <inertia  ixx="${2*mass*radius*radius/5}" ixy="0" ixz="0"
-              iyy="${2*mass*radius*radius/5}" iyz="0"
-              izz="${2*mass*radius*radius/5}" />
+    <inertia ixx="${2*mass*radius*radius/5}" ixy="0" ixz="0"
+             iyy="${2*mass*radius*radius/5}" iyz="0"
+             izz="${2*mass*radius*radius/5}" />
   </xacro:macro>
   <!-- Drive Wheel Macro -->
@@ -27,63 +27,47 @@
     <link name="${wheel_side}_wheel">
       <visual>
-        <origin xyz="0 0 0" rpy="0 0 0"/>
-        <geometry>
-          <cylinder length="${wheel_width}" radius="${wheel_radius}"/>
-        </geometry>
+        <geometry><cylinder length="${wheel_width}" radius="${wheel_radius}"/></geometry>
         <material name="black"/>
       </visual>
       <collision>
-        <origin xyz="0 0 0" rpy="0 0 0" />
-        <geometry>
-          <cylinder length="${wheel_width}" radius="${wheel_radius}"/>
-        </geometry>
+        <geometry><cylinder length="${wheel_width}" radius="${wheel_radius}"/></geometry>
       </collision>
       <inertial>
-        <origin xyz="0 0 0" />
         <mass value="${wheel_mass}" />
-        <inertia ixx="0.01300" ixy="0.0" ixz="0.0"
-                 iyy="0.007042" iyz="0.0"
-                 izz="0.007042" />
+        <inertia ixx="0.01300" ixy="0" ixz="0" iyy="0.007042" iyz="0" izz="0.007042" />
       </inertial>
-      <gazebo reference="${wheel_side}_wheel">
-        <mu1>10.0</mu1>
-        <mu2>10.0</mu2>
-        <kp>500000.0</kp>
-        <kd>10.0</kd>
-        <maxVel>1.1</maxVel>
-        <material>Gazebo/Black</material>
-      </gazebo>
     </link>
+    <gazebo reference="${wheel_side}_wheel">
+      <mu1>10.0</mu1>
+      <mu2>10.0</mu2>
+      <kp>500000.0</kp>
+      <kd>10.0</kd>
+      <maxVel>1.1</maxVel>
+      <material>Gazebo/Black</material>
+    </gazebo>
   </xacro:macro>
-  <!-- Front Caster Wheel Macro -->
-  <xacro:macro name="caster_front" params="caster_side offset_y">
-    <joint name="${caster_side}_caster_front_joint" type="fixed">
+  <!-- Passive Caster Wheel Macro -->
+  <xacro:macro name="caster" params="prefix offset_x offset_y mass:=5.2 mu1:=0.0 mu2:=0.0">
+    <joint name="${prefix}_caster_joint" type="fixed">
       <parent link="base_link"/>
-      <child link="${caster_side}_caster_front"/>
-      <origin xyz="0.650 ${offset_y} -0.109" rpy="0 0 0"/>
+      <child link="${prefix}_caster"/>
+      <origin xyz="${offset_x} ${offset_y} -0.109" rpy="0 0 0"/>
     </joint>
-    <link name="${caster_side}_caster_front">
+    <link name="${prefix}_caster">
       <visual>
-        <origin xyz="0 0 0" rpy="0 ${M_PI/2} 0" />
-        <geometry>
-          <sphere radius="${caster_radius}" />
-        </geometry>
+        <geometry><sphere radius="${caster_radius}" /></geometry>
         <material name="blue"/>
       </visual>
       <collision>
-        <origin xyz="0 0 0" rpy="0 ${M_PI/2} 0" />
-        <geometry>
-          <sphere radius="${caster_radius}"/>
-        </geometry>
+        <geometry><sphere radius="${caster_radius}"/></geometry>
       </collision>
       <inertial>
-        <origin xyz="0 0 0" rpy="0 ${M_PI/2} 0" />
-        <mass value="${caster_mass}"/>
-        <sphere_inertia mass="${caster_mass}" radius="${caster_radius}"/>
+        <mass value="${mass}"/>
+        <xacro:sphere_inertia mass="${mass}" radius="${caster_radius}"/>
       </inertial>
     </link>
-    <gazebo reference="${caster_side}_caster_front">
-      <mu1>0.0</mu1>
-      <mu2>0.0</mu2>
+    <gazebo reference="${prefix}_caster">
+      <mu1>${mu1}</mu1>
+      <mu2>${mu2}</mu2>
       <kp>1000000.0</kp>
       <kd>100.0</kd>
@@ -92,42 +76,57 @@
     </gazebo>
   </xacro:macro>
-  <!-- Back Caster Wheel Macro -->
-  <xacro:macro name="caster_back" params="caster_side offset_y">
-    <joint name="${caster_side}_caster_back_joint" type="fixed">
-      <parent link="base_link"/>
-      <child link="${caster_side}_caster_back"/>
-      <origin xyz="-0.650 ${offset_y} -0.109" rpy="0 0 0"/>
-      <axis xyz="0 0 1"/>
-    </joint>
-    <link name="${caster_side}_caster_back">
+  <!-- Cylindrical Laser Scanner Macro -->
+  <xacro:macro name="laser_sensor" params="name x y z roll pitch yaw mass:=0.5925 length:=0.151 radius:=0.05">
+    <link name="${name}_link">
       <visual>
-        <origin xyz="0 0 0" rpy="0 ${M_PI/2} 0" />
-        <geometry>
-          <sphere radius="${caster_radius}" />
-        </geometry>
+        <geometry><cylinder length="${length}" radius="${radius}"/></geometry>
         <material name="blue"/>
       </visual>
       <collision>
-        <origin xyz="0 0 0" rpy="0 ${M_PI/2} 0" />
-        <geometry>
-          <sphere radius="${caster_radius}" />
-        </geometry>
+        <geometry><cylinder length="${length}" radius="${radius}"/></geometry>
       </collision>
       <inertial>
-        <origin xyz="0 0 0.0" />
-        <mass value="0.01" />
-        <inertia ixx="0.001" ixy="0.0" ixz="0.0"
-                 iyy="0.001" iyz="0.0"
-                 izz="0.0001" />
+        <mass value="${mass}" />
+        <origin xyz="-7.88E-05 4.35E-05 -0.01694" rpy="0 0 0" />
+        <xacro:cylinder_inertia mass="${mass}" radius="${radius}" length="${length}"/>
       </inertial>
     </link>
-    <gazebo reference="${caster_side}_caster_back">
-      <mu1>1.0</mu1>
-      <mu2>1.0</mu2>
-      <kp>1000000.0</kp>
-      <kd>10.0</kd>
-      <maxVel>3.0</maxVel>
+    <joint name="${name}_joint" type="fixed">
+      <parent link="base_link"/>
+      <child link="${name}_link"/>
+      <origin xyz="${x} ${y} ${z}" rpy="${roll} ${pitch} ${yaw}"/>
+    </joint>
+    <gazebo reference="${name}_link">
       <material>Gazebo/Blue</material>
     </gazebo>
   </xacro:macro>
+  <!-- Camera Mount Joint, Visual Body, and Standard Optical Frame Macro -->
+  <xacro:macro name="camera_mount" params="num x y z roll pitch yaw">
+    <link name="camera_${num}_link">
+      <visual>
+        <geometry><box size="0.025 0.090 0.025"/></geometry>
+        <material name="black"/>
+      </visual>
+      <collision>
+        <geometry><box size="0.025 0.090 0.025"/></geometry>
+      </collision>
+      <inertial>
+        <mass value="0.1"/>
+        <origin xyz="0 0 0" rpy="0 0 0"/>
+        <xacro:box_inertia mass="0.1" size_x="0.025" size_y="0.090" size_z="0.025"/>
+      </inertial>
+    </link>
+    <joint name="camera_${num}_joint" type="fixed">
+      <parent link="base_link"/>
+      <child link="camera_${num}_link"/>
+      <origin xyz="${x} ${y} ${z}" rpy="${roll} ${pitch} ${yaw}"/>
+      <axis xyz="0 0 0"/>
+    </joint>
+    <link name="camera_${num}_color_optical_frame"/>
+    <joint name="camera_${num}_color_optical_joint" type="fixed">
+      <parent link="camera_${num}_link"/>
+      <child link="camera_${num}_color_optical_frame"/>
+      <origin xyz="0 0 0" rpy="-1.57 0 -1.57"/>
+    </joint>
+  </xacro:macro>
 </robot>

File: urdf/agv.urdf.xacro (robot description, xacro)
@@ -1,7 +1,4 @@
 <?xml version="1.0" ?>
 <robot name="agv" xmlns:xacro="http://ros.org/wiki/xacro">
-  <!-- General Arguments & Constants -->
-  <xacro:arg name="robot_namespace" default="/" />
-  <xacro:property name="M_PI" value="3.1415926535897931"/>
   <!-- Chassis Physical Dimensions & Mass -->
   <xacro:property name="chassis_length" value="1.558"/>
@@ -9,54 +6,30 @@
   <xacro:property name="chassis_height" value="0.280"/>
   <xacro:property name="chassis_mass" value="300"/>
-  <!-- Caster Wheel Physical Dimensions & Mass -->
+  <!-- Caster Wheel Dimensions -->
   <xacro:property name="caster_radius" value="0.062"/>
-  <xacro:property name="caster_length" value="0.05"/>
-  <xacro:property name="caster_mass" value="5.2"/>
-  <!-- Drive Wheel Physical Dimensions & Mass -->
+  <!-- Drive Wheel Dimensions -->
   <xacro:property name="wheel_width" value="0.05"/>
   <xacro:property name="wheel_radius" value="0.1"/>
   <xacro:property name="wheel_mass" value="2"/>
-  <!-- Path and Model Arguments -->
-  <xacro:arg name="config_path" default="" />
-  <xacro:arg name="robot_model" default="$(env AMR_MODEL)"/>
-  <xacro:arg name="parameters_dir" default="$(env ROS_PACKAGE_PATH)"/>
-  <!-- Included Xacro Files -->
-  <xacro:include filename="$(arg parameters_dir)/Product/$(arg robot_model)/RobotUrdf/common_properties.xacro"/>
-  <xacro:include filename="$(arg config_path)/_CONFIG_/laser_correction.xacro"/>
-  <xacro:include filename="$(arg config_path)/_CONFIG_/camera_correction.xacro"/>
-  <xacro:include filename="$(arg config_path)/_CONFIG_/imu_joint.xacro"/>
-  <xacro:include filename="$(arg parameters_dir)/Product/$(arg robot_model)/RobotUrdf/agv.gazebo.xacro"/>
-  <xacro:include filename="$(arg parameters_dir)/Product/$(arg robot_model)/RobotUrdf/agv.macros.xacro"/>
-  <!-- Base Footprint (Ground Projection Link) -->
+  <!-- Included Configurations & Modules -->
+  <xacro:include filename="config/common_properties.xacro"/>
+  <xacro:include filename="config/laser_correction.xacro"/>
+  <xacro:include filename="config/camera_correction.xacro"/>
+  <xacro:include filename="config/imu_joint.xacro"/>
+  <xacro:include filename="agv.gazebo.xacro"/>
+  <xacro:include filename="agv.macros.xacro"/>
+  <!-- Base Footprint & Link -->
   <link name="base_footprint"/>
   <joint name="base_footprint_to_base_link_joint" type="fixed">
     <parent link="base_footprint"/>
     <child link="base_link"/>
-    <origin xyz="0.0 0.0 0.0" rpy="0 0 0"/>
+    <origin xyz="0 0 0" rpy="0 0 0"/>
   </joint>
-  <!-- Chassis Base Link -->
   <link name="base_link">
-    <collision>
-      <origin xyz="0 0 0" rpy="0 0 0"/>
-      <geometry>
-        <box size="${chassis_length} ${chassis_width} ${chassis_height}"/>
-      </geometry>
-    </collision>
-    <visual>
-      <origin xyz="0 0 0" rpy="0 0 0"/>
-      <geometry>
-        <box size="${chassis_length} ${chassis_width} ${chassis_height}"/>
-      </geometry>
-      <material name="grey"/>
-    </visual>
+    <collision><geometry><box size="${chassis_length} ${chassis_width} ${chassis_height}"/></geometry></collision>
+    <visual><geometry><box size="${chassis_length} ${chassis_width} ${chassis_height}"/></geometry><material name="grey"/></visual>
     <inertial>
-      <origin xyz="0 0 0" />
       <mass value="${chassis_mass}" />
-      <inertia ixx="3.9687"
-        ixy="0.28534"
-        ixz="0.11898"
-        iyy="11.378"
-        iyz="0.0073517"
-        izz="8.1939" />
+      <inertia ixx="3.9687" ixy="0.28534" ixz="0.11898" iyy="11.378" iyz="0.00735" izz="8.1939" />
     </inertial>
   </link>
@@ -64,108 +37,20 @@
   <wheel wheel_side="left" offset_y="0.40649"/>
   <wheel wheel_side="right" offset_y="-0.40649"/>
-  <!-- Caster Wheels (Front & Back) -->
-  <caster_front caster_side="left" offset_y="0.400"/>
-  <caster_front caster_side="right" offset_y="-0.400"/>
-  <caster_back caster_side="left" offset_y="0.400" />
-  <caster_back caster_side="right" offset_y="-0.400"/>
-  <!-- Front Laser Scanner -->
-  <link name="laser_front_link">
+  <!-- Caster Wheels -->
+  <caster prefix="left_front" offset_x="0.650" offset_y="0.400" mass="5.2"/>
+  <caster prefix="right_front" offset_x="0.650" offset_y="-0.400" mass="5.2"/>
+  <caster prefix="left_back" offset_x="-0.650" offset_y="0.400" mass="0.01"/>
+  <caster prefix="right_back" offset_x="-0.650" offset_y="-0.400" mass="0.01"/>
+  <!-- Lasers -->
+  <laser_sensor name="laser_front" x="${laser_front_x}" y="${laser_front_y}" z="${laser_front_z}" roll="${laser_front_roll}" pitch="${laser_front_pitch}" yaw="${laser_front_yaw}"/>
+  <laser_sensor name="laser_back" x="${laser_back_x}" y="${laser_back_y}" z="${laser_back_z}" roll="${laser_back_roll}" pitch="${laser_back_pitch}" yaw="${laser_back_yaw}"/>
+  <laser_sensor name="laser_3d" x="${laser_3d_x}" y="${laser_3d_y}" z="${laser_3d_z}" roll="${laser_3d_roll}" pitch="${laser_3d_pitch}" yaw="${laser_3d_yaw}" mass="1.5"/>
+  <!-- IMU Sensor -->
+  <link name="imu_link">
     <visual>
-      <origin xyz="0.0 0.0 0.0" rpy="0 0 0"/>
-      <geometry>
-        <cylinder length="0.151" radius="0.05"/>
-      </geometry>
-      <material name="blue"/>
+      <geometry><box size="0.05 0.05 0.02"/></geometry>
+      <material name="black"/>
     </visual>
-    <collision>
-      <origin xyz="0.0 0.0 0.0" rpy="0 0 0"/>
-      <geometry>
-        <cylinder length="0.151" radius="0.05"/>
-      </geometry>
-    </collision>
-    <inertial>
-      <mass value="0.5925" />
-      <origin xyz="-7.8833E-05 4.3529E-05 -0.016941" rpy="0 0 0" />
-      <inertia ixx="0.00070857"
-        ixy="-1.3137E-06"
-        ixz="1.6001E-06"
-        iyy="0.00070663"
-        iyz="3.8031E-07"
-        izz="0.0008093" />
-    </inertial>
   </link>
-  <joint name="laser_front_joint" type="fixed">
-    <parent link="base_link"/>
-    <child link="laser_front_link"/>
-    <origin xyz="${laser_front_x} ${laser_front_y} ${laser_front_z}" rpy="${laser_front_roll} ${laser_front_pitch} ${laser_front_yaw}"/>
-  </joint>
-  <!-- Back Laser Scanner -->
-  <link name="laser_back_link">
-    <visual>
-      <origin xyz="0.0 0.0 0.0" rpy="0 0 0"/>
-      <geometry>
-        <cylinder length="0.151" radius="0.05"/>
-      </geometry>
-      <material name="blue"/>
-    </visual>
-    <collision>
-      <origin xyz="0.0 0.0 0.0" rpy="0 0 0"/>
-      <geometry>
-        <cylinder length="0.151" radius="0.05"/>
-      </geometry>
-    </collision>
-    <inertial>
-      <mass value="0.5925" />
-      <origin xyz="-7.8839E-05 4.3846E-05 -0.016941" rpy="0 0 0" />
-      <inertia ixx="0.00070857"
-        ixy="-1.3137E-06"
-        ixz="1.6001E-06"
-        iyy="0.00070663"
-        iyz="3.8031E-07"
-        izz="0.0008093"/>
-    </inertial>
-  </link>
-  <joint name="laser_back_joint" type="fixed">
-    <parent link="base_link"/>
-    <child link="laser_back_link"/>
-    <origin xyz="${laser_back_x} ${laser_back_y} ${laser_back_z}" rpy="${laser_back_roll} ${laser_back_pitch} ${laser_back_yaw}"/>
-  </joint>
-  <!-- 3D Laser Scanner -->
-  <link name="laser_3d_link">
-    <visual>
-      <origin xyz="0.0 0.0 0.0" rpy="0 0 0"/>
-      <geometry>
-        <cylinder length="0.151" radius="0.05"/>
-      </geometry>
-      <material name="blue"/>
-    </visual>
-    <collision>
-      <origin xyz="0.0 0.0 0.0" rpy="0 0 0"/>
-      <geometry>
-        <cylinder length="0.151" radius="0.05"/>
-      </geometry>
-    </collision>
-    <inertial>
-      <mass value="1.5" />
-      <origin xyz="0.0 0.0 0" />
-      <inertia ixx="0.003" ixy="0.0" ixz="0.0"
-               iyy="0.003" iyz="0.0"
-               izz="0.0018" />
-    </inertial>
-  </link>
-  <joint name="laser_3d_joint" type="fixed">
-    <parent link="base_link"/>
-    <child link="laser_3d_link"/>
-    <origin xyz="${laser_3d_x} ${laser_3d_y} ${laser_3d_z}" rpy="${laser_3d_roll} ${laser_3d_pitch} ${laser_3d_yaw}"/>
-  </joint>
-  <!-- Primary / PNF Laser Link -->
-  <link name="laser_pnf_link"/>
-  <joint name="laser_pnf_joint" type="fixed">
-    <parent link="base_link"/>
-    <child link="laser_pnf_link"/>
-    <origin xyz="${laser_x} ${laser_y} ${laser_z}" rpy="${laser_roll} ${laser_pitch} ${laser_yaw}"/>
-  </joint>
-  <!-- IMU Sensor -->
-  <link name="imu_link"/>
   <joint name="imu_joint" type="fixed">
     <parent link="base_link"/>
@@ -173,41 +58,8 @@
     <origin xyz="${imu_x} ${imu_y} ${imu_z}" rpy="${imu_roll} ${imu_pitch} ${imu_yaw}"/>
   </joint>
-  <!-- Camera 1 -->
-  <link name="camera_1_link"/>
-  <joint name="camera_1_joint" type="fixed">
-    <origin xyz="${camera_1_x} ${camera_1_y} ${camera_1_z}" rpy="${camera_1_roll} ${camera_1_pitch} ${camera_1_yaw}"/>
-    <parent link="base_link"/>
-    <child link="camera_1_link"/>
-    <axis xyz="0 0 0"/>
-  </joint>
-  <link name="camera_1_color_optical_frame"/>
-  <joint name="camera_1_color_optical_joint" type="fixed">
-    <parent link="camera_1_link"/>
-    <child link="camera_1_color_optical_frame"/>
-    <origin xyz="0.0 0.0 0.0" rpy="-1.57 0.0 -1.57"/>
-  </joint>
-  <!-- Camera 2 -->
-  <link name="camera_2_link"/>
-  <joint name="camera_2_joint" type="fixed">
-    <origin xyz="${camera_2_x} ${camera_2_y} ${camera_2_z}" rpy="${camera_2_roll} ${camera_2_pitch} ${camera_2_yaw}"/>
-    <parent link="base_link"/>
-    <child link="camera_2_link"/>
-    <axis xyz="0 0 0"/>
-  </joint>
-  <!-- Camera 3 -->
-  <link name="camera_3_link"/>
-  <joint name="camera_3_joint" type="fixed">
-    <origin xyz="${camera_3_x} ${camera_3_y} ${camera_3_z}" rpy="${camera_3_roll} ${camera_3_pitch} ${camera_3_yaw}"/>
-    <parent link="base_link"/>
-    <child link="camera_3_link"/>
-    <axis xyz="0 0 0"/>
-  </joint>
-  <!-- Camera 4 -->
-  <link name="camera_4_link"/>
-  <joint name="camera_4_joint" type="fixed">
-    <origin xyz="${camera_4_x} ${camera_4_y} ${camera_4_z}" rpy="${camera_4_roll} ${camera_4_pitch} ${camera_4_yaw}"/>
-    <parent link="base_link"/>
-    <child link="camera_4_link"/>
-    <axis xyz="0 0 0"/>
-  </joint>
+  <!-- Cameras (Mounts + Optical Frames) -->
+  <camera_mount num="1" x="${camera_1_x}" y="${camera_1_y}" z="${camera_1_z}" roll="${camera_1_roll}" pitch="${camera_1_pitch}" yaw="${camera_1_yaw}"/>
+  <camera_mount num="2" x="${camera_2_x}" y="${camera_2_y}" z="${camera_2_z}" roll="${camera_2_roll}" pitch="${camera_2_pitch}" yaw="${camera_2_yaw}"/>
+  <camera_mount num="3" x="${camera_3_x}" y="${camera_3_y}" z="${camera_3_z}" roll="${camera_3_roll}" pitch="${camera_3_pitch}" yaw="${camera_3_yaw}"/>
+  <camera_mount num="4" x="${camera_4_x}" y="${camera_4_y}" z="${camera_4_z}" roll="${camera_4_roll}" pitch="${camera_4_pitch}" yaw="${camera_4_yaw}"/>
 </robot>
