Commit message: A2: modified urd files for modularity

File: urdf/config/laser_correction.xacro (robot description, xacro)
@@ -1,15 +1,19 @@
-<robot name="agv_trial" xmlns:xacro="http://ros.org/wiki/xacro">
-  <xacro:property name="laser_front_x" value="0.71179" /> <!-- 0.70179 -->
-  <xacro:property name="laser_front_y" value="0.47912" /> <!-- 0.39912 -->
+<?xml version="1.0" ?>
+<robot name="agv" xmlns:xacro="http://ros.org/wiki/xacro">
+  <!-- Front Laser Calibration Offsets -->
+  <xacro:property name="laser_front_x" value="0.71179" />
+  <xacro:property name="laser_front_y" value="0.47912" />
   <xacro:property name="laser_front_z" value="0.17501" />
   <xacro:property name="laser_front_roll" value="-3.1416" />
   <xacro:property name="laser_front_pitch" value="0.0" />
-  <xacro:property name="laser_front_yaw" value="0.768395" /> <!-- 0.7854 -->
+  <xacro:property name="laser_front_yaw" value="0.768395" />
+  <!-- Back Laser Calibration Offsets -->
   <xacro:property name="laser_back_x" value="-0.70179" />
-  <xacro:property name="laser_back_y" value="-0.30912" /> <!-- -0.39912 -->
+  <xacro:property name="laser_back_y" value="-0.30912" />
   <xacro:property name="laser_back_z" value="0.17501" />
   <xacro:property name="laser_back_roll" value="-3.1416" />
   <xacro:property name="laser_back_pitch" value="0.0" />
-  <xacro:property name="laser_back_yaw" value="-2.33875" /> <!-- -2.3562 -->
+  <xacro:property name="laser_back_yaw" value="-2.33875" />
+  <!-- 3D Laser Calibration Offsets -->
   <xacro:property name="laser_3d_x" value="0.82726" />
   <xacro:property name="laser_3d_y" value="-0.55936" />

Commit message: A3: updated gz sim and modified xacro files

File: urdf/agv.gazebo.xacro (robot description, xacro)
@@ -1,124 +1,56 @@
 <?xml version="1.0"?>
 <robot name="agv" xmlns:xacro="http://ros.org/wiki/xacro">
-  <xacro:arg name="laser_visual" default="true"/>
-  <xacro:arg name="imu_visual"   default="true"/>
-  <!-- Differential Drive Controller Plugin -->
+  <xacro:arg name="imu_visual" default="false"/>
+  <!-- System Plugins -->
   <gazebo>
-    <plugin name="differential_drive_controller" filename="libgazebo_ros_diff_drive.so">
-      <commandTopic>cmd_vel</commandTopic>
-      <rosDebugLevel>Debug</rosDebugLevel>
-      <odometryTopic>odom</odometryTopic>
-      <odometryFrame>odom</odometryFrame>
-      <robotBaseFrame>base_footprint</robotBaseFrame>
-      <publishWheelTF>false</publishWheelTF>
-      <publishWheelJointState>true</publishWheelJointState>
-      <legacyMode>false</legacyMode>
-      <updateRate>50</updateRate>
-      <alwaysOn>true</alwaysOn>
-      <leftJoint>left_wheel_joint</leftJoint>
-      <rightJoint>right_wheel_joint</rightJoint>
-      <wheelSeparation>0.81298</wheelSeparation>
-      <wheelDiameter>0.200</wheelDiameter>
-      <wheelAcceleration>1</wheelAcceleration>
-      <wheelTorque>34.52</wheelTorque>
+    <!-- Diff Drive -->
+    <plugin filename="gz-sim-diff-drive-system" name="gz::sim::systems::DiffDrive">
+      <left_joint>left_wheel_joint</left_joint>
+      <right_joint>right_wheel_joint</right_joint>
+      <wheel_separation>${wheel_track}</wheel_separation>
+      <wheel_radius>${wheel_radius}</wheel_radius>
+      <max_linear_acceleration>1.0</max_linear_acceleration>
+      <max_angular_acceleration>2.0</max_angular_acceleration>
+      <min_velocity>-1.5</min_velocity>
+      <max_velocity>1.5</max_velocity>
+      <topic>/cmd_vel</topic>
+      <odom_topic>/odom</odom_topic>
+      <frame_id>odom</frame_id>
+      <child_frame_id>base_footprint</child_frame_id>
+      <odom_publisher_frequency>50</odom_publisher_frequency>
+      <tf_topic>/tf</tf_topic>
+    </plugin>
+    <!-- Joint State Publisher -->
+    <plugin filename="gz-sim-joint-state-publisher-system" name="gz::sim::systems::JointStatePublisher">
+      <topic>/joint_states</topic>
+      <joint_name>left_wheel_joint</joint_name>
+      <joint_name>right_wheel_joint</joint_name>
     </plugin>
   </gazebo>
+  <!-- Base Link Material -->
   <gazebo reference="base_link">
     <material>Gazebo/Grey</material>
   </gazebo>
-  <!-- Drive Wheel Contact Properties -->
-  <gazebo reference="left_wheel">
-    <mu1>1000000.0</mu1>
-    <mu2>100000.0</mu2>
-    <kp>5000000.0</kp>
-    <kd>100.0</kd>
-    <minDepth>0.001</minDepth>
-    <maxVel>1.5</maxVel>
-    <fdir1>1 0 0</fdir1>
-    <material>Gazebo/Grey</material>
+  <!-- IMU Sensor (Standard ROS topic: /imu/data, tune noise stddev via Allan variance/datasheet) -->
+  <gazebo reference="imu_link">
+    <sensor name="imu_sensor" type="imu">
+      <always_on>true</always_on>
+      <update_rate>100.0</update_rate>
+      <visualize>$(arg imu_visual)</visualize>
+      <topic>/imu/data</topic>
+      <gz_frame_id>imu_link</gz_frame_id>
+      <imu>
+        <angular_velocity>
+          <x><noise type="gaussian"><mean>0.0</mean><stddev>2e-4</stddev></noise></x>
+          <y><noise type="gaussian"><mean>0.0</mean><stddev>2e-4</stddev></noise></y>
+          <z><noise type="gaussian"><mean>0.0</mean><stddev>2e-4</stddev></noise></z>
+        </angular_velocity>
+        <linear_acceleration>
+          <x><noise type="gaussian"><mean>0.0</mean><stddev>1.7e-2</stddev></noise></x>
+          <y><noise type="gaussian"><mean>0.0</mean><stddev>1.7e-2</stddev></noise></y>
+          <z><noise type="gaussian"><mean>0.0</mean><stddev>1.7e-2</stddev></noise></z>
+        </linear_acceleration>
+      </imu>
+    </sensor>
   </gazebo>
-  <gazebo reference="right_wheel">
-    <mu1>1000000.0</mu1>
-    <mu2>100000.0</mu2>
-    <kp>5000000.0</kp>
-    <kd>100.0</kd>
-    <minDepth>0.001</minDepth>
-    <maxVel>0.8</maxVel>
-    <fdir1>1 0 0</fdir1>
-    <material>Gazebo/Grey</material>
-  </gazebo>
-  <!-- IMU Sensor Plugin -->
-  <gazebo>
-    <plugin name="imu_sensor_plugin" filename="libgazebo_ros_imu.so">
-      <alwaysOn>true</alwaysOn>
-      <bodyName>imu_link</bodyName>
-      <topicName>imu</topicName>
-      <serviceName>imu_service</serviceName>
-      <gaussianNoise>0.0</gaussianNoise>
-      <updateRate>100.0</updateRate>
-      <imu>
-        <noise>
-          <type>gaussian</type>
-          <rate>
-            <mean>0.0</mean>
-            <stddev>2e-4</stddev>
-            <bias_mean>0.0000075</bias_mean>
-            <bias_stddev>0.0000008</bias_stddev>
-          </rate>
-          <accel>
-            <mean>0.0</mean>
-            <stddev>1.7e-2</stddev>
-            <bias_mean>0.1</bias_mean>
-            <bias_stddev>0.001</bias_stddev>
-          </accel>
-        </noise>
-      </imu>
-    </plugin>
-  </gazebo>
-  <gazebo reference="imu_link">
-    <sensor type="imu" name="imu_sensor">
-      <always_on>true</always_on>
-      <update_rate>100</update_rate>
-      <visualize>$(arg imu_visual)</visualize>
-    </sensor>
-    <material>Gazebo/Grey</material>
-  </gazebo>
-  <!-- Laser Sensor Plugin Macro -->
-  <xacro:macro name="gazebo_laser_plugin" params="link_name sensor_name topic_name update_rate:=18.0 min_angle:=-3.14159 max_angle:=3.14159">
-    <gazebo reference="${link_name}">
-      <material>Gazebo/Blue</material>
-      <sensor type="ray" name="${sensor_name}">
-        <pose>0 0 0 0 0 0</pose>
-        <visualize>$(arg laser_visual)</visualize>
-        <update_rate>${update_rate}</update_rate>
-        <ray>
-          <scan>
-            <horizontal>
-              <samples>360</samples>
-              <resolution>1</resolution>
-              <min_angle>${min_angle}</min_angle>
-              <max_angle>${max_angle}</max_angle>
-            </horizontal>
-          </scan>
-          <range>
-            <min>0.120</min>
-            <max>10.0</max>
-            <resolution>0.025</resolution>
-          </range>
-          <noise>
-            <type>gaussian</type>
-            <mean>0.0</mean>
-            <stddev>0.01</stddev>
-          </noise>
-        </ray>
-        <plugin name="${sensor_name}_controller" filename="libgazebo_ros_laser.so">
-          <topicName>${topic_name}</topicName>
-          <frameName>${link_name}</frameName>
-        </plugin>
-      </sensor>
-    </gazebo>
-  </xacro:macro>
-  <!-- Front and Back 2D Laser Ray Sensors -->
-  <xacro:gazebo_laser_plugin link_name="laser_front_link" sensor_name="front_laser" topic_name="scan_front"/>
-  <xacro:gazebo_laser_plugin link_name="laser_back_link"  sensor_name="back_laser"  topic_name="scan_back"/>
 </robot>

File: urdf/agv.macros.xacro (robot description, xacro)
@@ -10,5 +10,5 @@
     <inertia  ixx="${mass*(size_y*size_y + size_z*size_z)/12}" ixy="0" ixz="0"
               iyy="${mass*(size_x*size_x + size_z*size_z)/12}" iyz="0"
-              izz="${mass*(size_x*size_x + size_z*size_z)/12}" />
+              izz="${mass*(size_x*size_x + size_y*size_y)/12}" />
   </xacro:macro>
   <xacro:macro name="sphere_inertia" params="mass radius">
@@ -35,5 +35,5 @@
       <inertial>
         <mass value="${wheel_mass}" />
-        <inertia ixx="0.01300" ixy="0" ixz="0" iyy="0.007042" iyz="0" izz="0.007042" />
+        <xacro:cylinder_inertia mass="${wheel_mass}" radius="${wheel_radius}" length="${wheel_width}"/>
       </inertial>
     </link>
@@ -47,5 +47,5 @@
     </gazebo>
   </xacro:macro>
-  <!-- Passive Caster Wheel Macro -->
+  <!-- Single Passive Caster Macro -->
   <xacro:macro name="caster" params="prefix offset_x offset_y mass:=5.2 mu1:=0.0 mu2:=0.0">
     <joint name="${prefix}_caster_joint" type="fixed">
@@ -76,6 +76,11 @@
     </gazebo>
   </xacro:macro>
-  <!-- Cylindrical Laser Scanner Macro -->
-  <xacro:macro name="laser_sensor" params="name x y z roll pitch yaw mass:=0.5925 length:=0.151 radius:=0.05">
+  <!-- Symmetric Caster Pair Macro (Left & Right) -->
+  <xacro:macro name="caster_pair" params="location offset_x offset_y mass:=5.2">
+    <xacro:caster prefix="left_${location}"  offset_x="${offset_x}" offset_y="${offset_y}"  mass="${mass}"/>
+    <xacro:caster prefix="right_${location}" offset_x="${offset_x}" offset_y="${-offset_y}" mass="${mass}"/>
+  </xacro:macro>
+  <!-- Self-Contained Cylindrical LiDAR Macro (Kinematics + Gz Sim Sensor Stream) -->
+  <xacro:macro name="lidar_sensor" params="name x y z roll pitch yaw topic_name mass:=0.5925 length:=0.151 radius:=0.05 samples:=360 v_samples:=1 min_angle:=-3.14159 max_angle:=3.14159 v_min_angle:=-0.261799 v_max_angle:=0.261799 min_range:=0.120 max_range:=15.0 update_rate:=20.0 noise_stddev:=0.01">
     <link name="${name}_link">
       <visual>
@@ -97,11 +102,47 @@
       <origin xyz="${x} ${y} ${z}" rpy="${roll} ${pitch} ${yaw}"/>
     </joint>
+    <!-- Encapsulated Gz Sim LiDAR Sensor -->
     <gazebo reference="${name}_link">
       <material>Gazebo/Blue</material>
+      <sensor name="${name}_sensor" type="gpu_lidar">
+        <always_on>true</always_on>
+        <update_rate>${update_rate}</update_rate>
+        <visualize>false</visualize>
+        <topic>${topic_name}</topic>
+        <gz_frame_id>${name}_link</gz_frame_id>
+        <lidar>
+          <scan>
+            <horizontal>
+              <samples>${samples}</samples>
+              <resolution>1</resolution>
+              <min_angle>${min_angle}</min_angle>
+              <max_angle>${max_angle}</max_angle>
+            </horizontal>
+            <xacro:if value="${v_samples > 1}">
+              <vertical>
+                <samples>${v_samples}</samples>
+                <resolution>1</resolution>
+                <min_angle>${v_min_angle}</min_angle>
+                <max_angle>${v_max_angle}</max_angle>
+              </vertical>
+            </xacro:if>
+          </scan>
+          <range>
+            <min>${min_range}</min>
+            <max>${max_range}</max>
+            <resolution>0.015</resolution>
+          </range>
+          <noise>
+            <type>gaussian</type>
+            <mean>0.0</mean>
+            <stddev>${noise_stddev}</stddev>
+          </noise>
+        </lidar>
+      </sensor>
     </gazebo>
   </xacro:macro>
-  <!-- Camera Mount Joint, Visual Body, and Standard Optical Frame Macro -->
-  <xacro:macro name="camera_mount" params="num x y z roll pitch yaw">
-    <link name="camera_${num}_link">
+  <!-- Self-Contained Camera Macro (Kinematics + Optical Frame + Gz Sim Stream) -->
+  <xacro:macro name="camera_mount" params="name x y z roll pitch yaw width:=640 height:=480 hfov:=1.5184 update_rate:=30.0">
+    <link name="${name}_link">
       <visual>
         <geometry><box size="0.025 0.090 0.025"/></geometry>
@@ -117,16 +158,38 @@
       </inertial>
     </link>
-    <joint name="camera_${num}_joint" type="fixed">
+    <joint name="${name}_joint" type="fixed">
       <parent link="base_link"/>
-      <child link="camera_${num}_link"/>
+      <child link="${name}_link"/>
       <origin xyz="${x} ${y} ${z}" rpy="${roll} ${pitch} ${yaw}"/>
       <axis xyz="0 0 0"/>
     </joint>
-    <link name="camera_${num}_color_optical_frame"/>
-    <joint name="camera_${num}_color_optical_joint" type="fixed">
-      <parent link="camera_${num}_link"/>
-      <child link="camera_${num}_color_optical_frame"/>
+    <link name="${name}_color_optical_frame"/>
+    <joint name="${name}_color_optical_joint" type="fixed">
+      <parent link="${name}_link"/>
+      <child link="${name}_color_optical_frame"/>
       <origin xyz="0 0 0" rpy="-1.57 0 -1.57"/>
     </joint>
+    <!-- Encapsulated Gz Sim Camera Sensor -->
+    <gazebo reference="${name}_link">
+      <sensor name="${name}" type="camera">
+        <always_on>true</always_on>
+        <update_rate>${update_rate}</update_rate>
+        <visualize>false</visualize>
+        <topic>/${name}/image_raw</topic>
+        <gz_frame_id>${name}_color_optical_frame</gz_frame_id>
+        <camera>
+          <horizontal_fov>${hfov}</horizontal_fov>
+          <image>
+            <width>${width}</width>
+            <height>${height}</height>
+            <format>R8G8B8</format>
+          </image>
+          <clip>
+            <near>0.1</near>
+            <far>15.0</far>
+          </clip>
+        </camera>
+      </sensor>
+    </gazebo>
   </xacro:macro>
 </robot>

File: urdf/agv.urdf.xacro (robot description, xacro)
@@ -8,15 +8,16 @@
   <!-- Caster Wheel Dimensions -->
   <xacro:property name="caster_radius" value="0.062"/>
-  <!-- Drive Wheel Dimensions -->
+  <!-- Drive Wheel Dimensions & Kinematics -->
   <xacro:property name="wheel_width" value="0.05"/>
   <xacro:property name="wheel_radius" value="0.1"/>
   <xacro:property name="wheel_mass" value="2"/>
+  <xacro:property name="wheel_track" value="0.81298"/>
   <!-- Included Configurations & Modules -->
   <xacro:include filename="config/common_properties.xacro"/>
-  <xacro:include filename="config/laser_correction.xacro"/>
+  <xacro:include filename="config/lidar_correction.xacro"/>
   <xacro:include filename="config/camera_correction.xacro"/>
   <xacro:include filename="config/imu_joint.xacro"/>
+  <xacro:include filename="agv.macros.xacro"/>
   <xacro:include filename="agv.gazebo.xacro"/>
-  <xacro:include filename="agv.macros.xacro"/>
   <!-- Base Footprint & Link -->
   <link name="base_footprint"/>
@@ -34,16 +35,14 @@
     </inertial>
   </link>
-  <!-- Drive Wheels -->
-  <wheel wheel_side="left" offset_y="0.40649"/>
-  <wheel wheel_side="right" offset_y="-0.40649"/>
-  <!-- Caster Wheels -->
-  <caster prefix="left_front" offset_x="0.650" offset_y="0.400" mass="5.2"/>
-  <caster prefix="right_front" offset_x="0.650" offset_y="-0.400" mass="5.2"/>
-  <caster prefix="left_back" offset_x="-0.650" offset_y="0.400" mass="0.01"/>
-  <caster prefix="right_back" offset_x="-0.650" offset_y="-0.400" mass="0.01"/>
-  <!-- Lasers -->
-  <laser_sensor name="laser_front" x="${laser_front_x}" y="${laser_front_y}" z="${laser_front_z}" roll="${laser_front_roll}" pitch="${laser_front_pitch}" yaw="${laser_front_yaw}"/>
-  <laser_sensor name="laser_back" x="${laser_back_x}" y="${laser_back_y}" z="${laser_back_z}" roll="${laser_back_roll}" pitch="${laser_back_pitch}" yaw="${laser_back_yaw}"/>
-  <laser_sensor name="laser_3d" x="${laser_3d_x}" y="${laser_3d_y}" z="${laser_3d_z}" roll="${laser_3d_roll}" pitch="${laser_3d_pitch}" yaw="${laser_3d_yaw}" mass="1.5"/>
+  <!-- Drive Wheels (Symmetric Mounting based on wheel_track) -->
+  <wheel wheel_side="left"  offset_y="${wheel_track / 2}"/>
+  <wheel wheel_side="right" offset_y="${-wheel_track / 2}"/>
+  <!-- Caster Wheel Pairs (Front & Back) -->
+  <caster_pair location="front" offset_x="0.650"  offset_y="0.400" mass="5.2"/>
+  <caster_pair location="back"  offset_x="-0.650" offset_y="0.400" mass="0.01"/>
+  <!-- 2D & 3D LiDAR Sensors (Kinematics + Simulation Stream) -->
+  <lidar_sensor name="front_lidar" x="${front_lidar_x}" y="${front_lidar_y}" z="${front_lidar_z}" roll="${front_lidar_roll}" pitch="${front_lidar_pitch}" yaw="${front_lidar_yaw}" topic_name="/front_lidar/scan"/>
+  <lidar_sensor name="rear_lidar"  x="${rear_lidar_x}"  y="${rear_lidar_y}"  z="${rear_lidar_z}"  roll="${rear_lidar_roll}"  pitch="${rear_lidar_pitch}"  yaw="${rear_lidar_yaw}"  topic_name="/rear_lidar/scan"/>
+  <lidar_sensor name="lidar_3d"    x="${lidar_3d_x}"    y="${lidar_3d_y}"    z="${lidar_3d_z}"    roll="${lidar_3d_roll}"    pitch="${lidar_3d_pitch}"    yaw="${lidar_3d_yaw}"    topic_name="/lidar_3d/points" mass="1.5" samples="1800" v_samples="16" v_min_angle="-0.261799" v_max_angle="0.261799" min_range="0.20" max_range="50.0" update_rate="10.0" noise_stddev="0.02"/>
   <!-- IMU Sensor -->
   <link name="imu_link">
@@ -58,8 +57,8 @@
     <origin xyz="${imu_x} ${imu_y} ${imu_z}" rpy="${imu_roll} ${imu_pitch} ${imu_yaw}"/>
   </joint>
-  <!-- Cameras (Mounts + Optical Frames) -->
-  <camera_mount num="1" x="${camera_1_x}" y="${camera_1_y}" z="${camera_1_z}" roll="${camera_1_roll}" pitch="${camera_1_pitch}" yaw="${camera_1_yaw}"/>
-  <camera_mount num="2" x="${camera_2_x}" y="${camera_2_y}" z="${camera_2_z}" roll="${camera_2_roll}" pitch="${camera_2_pitch}" yaw="${camera_2_yaw}"/>
-  <camera_mount num="3" x="${camera_3_x}" y="${camera_3_y}" z="${camera_3_z}" roll="${camera_3_roll}" pitch="${camera_3_pitch}" yaw="${camera_3_yaw}"/>
-  <camera_mount num="4" x="${camera_4_x}" y="${camera_4_y}" z="${camera_4_z}" roll="${camera_4_roll}" pitch="${camera_4_pitch}" yaw="${camera_4_yaw}"/>
+  <!-- Cameras (Mounts + Optical Frames + Simulation Stream) -->
+  <camera_mount name="camera_front_left"  x="${camera_front_left_x}"  y="${camera_front_left_y}"  z="${camera_front_left_z}"  roll="${camera_front_left_roll}"  pitch="${camera_front_left_pitch}"  yaw="${camera_front_left_yaw}"/>
+  <camera_mount name="camera_front_right" x="${camera_front_right_x}" y="${camera_front_right_y}" z="${camera_front_right_z}" roll="${camera_front_right_roll}" pitch="${camera_front_right_pitch}" yaw="${camera_front_right_yaw}"/>
+  <camera_mount name="camera_rear_left"   x="${camera_rear_left_x}"   y="${camera_rear_left_y}"   z="${camera_rear_left_z}"   roll="${camera_rear_left_roll}"   pitch="${camera_rear_left_pitch}"   yaw="${camera_rear_left_yaw}"/>
+  <camera_mount name="camera_rear_right"  x="${camera_rear_right_x}"  y="${camera_rear_right_y}"  z="${camera_rear_right_z}"  roll="${camera_rear_right_roll}"  pitch="${camera_rear_right_pitch}"  yaw="${camera_rear_right_yaw}"/>
 </robot>

File: urdf/config/camera_correction.xacro (robot description, xacro)
@@ -1,31 +1,31 @@
 <?xml version="1.0" ?>
 <robot name="agv" xmlns:xacro="http://ros.org/wiki/xacro">
-  <!-- Camera 1 Mount Offsets -->
-  <xacro:property name="camera_1_x" value="0.73448"/>
-  <xacro:property name="camera_1_y" value="0.1567"/>
-  <xacro:property name="camera_1_z" value="0.1225"/>
-  <xacro:property name="camera_1_roll" value="0.0"/>
-  <xacro:property name="camera_1_pitch" value="0.0"/>
-  <xacro:property name="camera_1_yaw" value="-0.5236"/>
-  <!-- Camera 2 Mount Offsets -->
-  <xacro:property name="camera_2_x" value="0.73448"/>
-  <xacro:property name="camera_2_y" value="-0.1567"/>
-  <xacro:property name="camera_2_z" value="0.1225"/>
-  <xacro:property name="camera_2_roll" value="0.0"/>
-  <xacro:property name="camera_2_pitch" value="0.0"/>
-  <xacro:property name="camera_2_yaw" value="0.5236"/>
-  <!-- Camera 3 Mount Offsets -->
-  <xacro:property name="camera_3_x" value="-0.73558"/>
-  <xacro:property name="camera_3_y" value="-0.1568"/>
-  <xacro:property name="camera_3_z" value="0.1225"/>
-  <xacro:property name="camera_3_roll" value="0.0"/>
-  <xacro:property name="camera_3_pitch" value="0.0"/>
-  <xacro:property name="camera_3_yaw" value="2.618"/>
-  <!-- Camera 4 Mount Offsets -->
-  <xacro:property name="camera_4_x" value="-0.73558"/>
-  <xacro:property name="camera_4_y" value="0.1568"/>
-  <xacro:property name="camera_4_z" value="0.1225"/>
-  <xacro:property name="camera_4_roll" value="0.0"/>
-  <xacro:property name="camera_4_pitch" value="0.0"/>
-  <xacro:property name="camera_4_yaw" value="-2.618"/>
+  <!-- Front Left Camera Mount Offsets -->
+  <xacro:property name="camera_front_left_x" value="0.73448"/>
+  <xacro:property name="camera_front_left_y" value="0.1567"/>
+  <xacro:property name="camera_front_left_z" value="0.1225"/>
+  <xacro:property name="camera_front_left_roll" value="0.0"/>
+  <xacro:property name="camera_front_left_pitch" value="0.0"/>
+  <xacro:property name="camera_front_left_yaw" value="-0.5236"/>
+  <!-- Front Right Camera Mount Offsets -->
+  <xacro:property name="camera_front_right_x" value="0.73448"/>
+  <xacro:property name="camera_front_right_y" value="-0.1567"/>
+  <xacro:property name="camera_front_right_z" value="0.1225"/>
+  <xacro:property name="camera_front_right_roll" value="0.0"/>
+  <xacro:property name="camera_front_right_pitch" value="0.0"/>
+  <xacro:property name="camera_front_right_yaw" value="0.5236"/>
+  <!-- Rear Left Camera Mount Offsets -->
+  <xacro:property name="camera_rear_left_x" value="-0.73558"/>
+  <xacro:property name="camera_rear_left_y" value="0.1568"/>
+  <xacro:property name="camera_rear_left_z" value="0.1225"/>
+  <xacro:property name="camera_rear_left_roll" value="0.0"/>
+  <xacro:property name="camera_rear_left_pitch" value="0.0"/>
+  <xacro:property name="camera_rear_left_yaw" value="-2.618"/>
+  <!-- Rear Right Camera Mount Offsets -->
+  <xacro:property name="camera_rear_right_x" value="-0.73558"/>
+  <xacro:property name="camera_rear_right_y" value="-0.1568"/>
+  <xacro:property name="camera_rear_right_z" value="0.1225"/>
+  <xacro:property name="camera_rear_right_roll" value="0.0"/>
+  <xacro:property name="camera_rear_right_pitch" value="0.0"/>
+  <xacro:property name="camera_rear_right_yaw" value="2.618"/>
 </robot>
