Commit message: A4: Final URDF

File: urdf/agv.macros.xacro (robot description, xacro)
@@ -22,5 +22,5 @@
       <parent link="base_link"/>
       <child link="${wheel_side}_wheel"/>
-      <origin xyz="0.0 ${offset_y} -0.04625" rpy="-1.57 0 0"/>
+      <origin xyz="0.0 ${offset_y} ${wheel_offset_z}" rpy="-1.57 0 0"/>
       <axis xyz="0 0 1"/>
     </joint>
@@ -48,9 +48,9 @@
   </xacro:macro>
   <!-- Single Passive Caster Macro -->
-  <xacro:macro name="caster" params="prefix offset_x offset_y mass:=5.2 mu1:=0.0 mu2:=0.0">
+  <xacro:macro name="caster" params="prefix offset_x offset_y mass:=${caster_mass} mu1:=0.0 mu2:=0.0">
     <joint name="${prefix}_caster_joint" type="fixed">
       <parent link="base_link"/>
       <child link="${prefix}_caster"/>
-      <origin xyz="${offset_x} ${offset_y} -0.109" rpy="0 0 0"/>
+      <origin xyz="${offset_x} ${offset_y} ${caster_offset_z}" rpy="0 0 0"/>
     </joint>
     <link name="${prefix}_caster">
@@ -77,10 +77,10 @@
   </xacro:macro>
   <!-- Symmetric Caster Pair Macro (Left & Right) -->
-  <xacro:macro name="caster_pair" params="location offset_x offset_y mass:=5.2">
+  <xacro:macro name="caster_pair" params="location offset_x offset_y mass:=${caster_mass}">
     <xacro:caster prefix="left_${location}"  offset_x="${offset_x}" offset_y="${offset_y}"  mass="${mass}"/>
     <xacro:caster prefix="right_${location}" offset_x="${offset_x}" offset_y="${-offset_y}" mass="${mass}"/>
   </xacro:macro>
   <!-- Self-Contained Cylindrical LiDAR Macro (Kinematics + Gz Sim Sensor Stream) -->
-  <xacro:macro name="lidar_sensor" params="name x y z roll pitch yaw topic_name mass:=0.5925 length:=0.151 radius:=0.05 samples:=360 v_samples:=1 min_angle:=-3.14159 max_angle:=3.14159 v_min_angle:=-0.261799 v_max_angle:=0.261799 min_range:=0.120 max_range:=15.0 update_rate:=20.0 noise_stddev:=0.01">
+  <xacro:macro name="lidar_sensor" params="name x y z roll pitch yaw topic_name mass:=0.5925 length:=0.151 radius:=0.05 samples:=360 v_samples:=1 h_resolution:=1 v_resolution:=1 min_angle:=-3.14159 max_angle:=3.14159 v_min_angle:=-0.261799 v_max_angle:=0.261799 min_range:=0.120 max_range:=15.0 range_resolution:=0.01 update_rate:=20.0 noise_stddev:=0.01">
     <link name="${name}_link">
       <visual>
@@ -115,5 +115,5 @@
             <horizontal>
               <samples>${samples}</samples>
-              <resolution>1</resolution>
+              <resolution>${h_resolution}</resolution>
               <min_angle>${min_angle}</min_angle>
               <max_angle>${max_angle}</max_angle>
@@ -122,5 +122,5 @@
               <vertical>
                 <samples>${v_samples}</samples>
-                <resolution>1</resolution>
+                <resolution>${v_resolution}</resolution>
                 <min_angle>${v_min_angle}</min_angle>
                 <max_angle>${v_max_angle}</max_angle>
@@ -131,5 +131,5 @@
             <min>${min_range}</min>
             <max>${max_range}</max>
-            <resolution>0.015</resolution>
+            <resolution>${range_resolution}</resolution>
           </range>
           <noise>
@@ -162,5 +162,4 @@
       <child link="${name}_link"/>
       <origin xyz="${x} ${y} ${z}" rpy="${roll} ${pitch} ${yaw}"/>
-      <axis xyz="0 0 0"/>
     </joint>
     <link name="${name}_color_optical_frame"/>

File: urdf/agv.urdf.xacro (robot description, xacro)
@@ -1,18 +1,7 @@
 <?xml version="1.0" ?>
 <robot name="agv" xmlns:xacro="http://ros.org/wiki/xacro">
-  <!-- Chassis Physical Dimensions & Mass -->
-  <xacro:property name="chassis_length" value="1.558"/>
-  <xacro:property name="chassis_width" value="0.965"/>
-  <xacro:property name="chassis_height" value="0.280"/>
-  <xacro:property name="chassis_mass" value="300"/>
-  <!-- Caster Wheel Dimensions -->
-  <xacro:property name="caster_radius" value="0.062"/>
-  <!-- Drive Wheel Dimensions & Kinematics -->
-  <xacro:property name="wheel_width" value="0.05"/>
-  <xacro:property name="wheel_radius" value="0.1"/>
-  <xacro:property name="wheel_mass" value="2"/>
-  <xacro:property name="wheel_track" value="0.81298"/>
-  <!-- Included Configurations & Modules -->
+  <!-- Configurations & Parameters -->
   <xacro:include filename="config/common_properties.xacro"/>
+  <xacro:include filename="config/robot_dimensions.xacro"/>
   <xacro:include filename="config/lidar_correction.xacro"/>
   <xacro:include filename="config/camera_correction.xacro"/>
@@ -20,14 +9,15 @@
   <xacro:include filename="agv.macros.xacro"/>
   <xacro:include filename="agv.gazebo.xacro"/>
-  <!-- Base Footprint & Link -->
+  <!-- Base Footprint (Ground Plane Z=0) to Base Link Elevation -->
   <link name="base_footprint"/>
   <joint name="base_footprint_to_base_link_joint" type="fixed">
     <parent link="base_footprint"/>
     <child link="base_link"/>
-    <origin xyz="0 0 0" rpy="0 0 0"/>
+    <origin xyz="0 0 ${-ground_contact_z}" rpy="0 0 0"/>
   </joint>
   <link name="base_link">
     <collision><geometry><box size="${chassis_length} ${chassis_width} ${chassis_height}"/></geometry></collision>
     <visual><geometry><box size="${chassis_length} ${chassis_width} ${chassis_height}"/></geometry><material name="grey"/></visual>
+    <!-- Measured/CAD empirical mass matrix including internal battery/payload asymmetry -->
     <inertial>
       <mass value="${chassis_mass}" />
@@ -39,6 +29,6 @@
   <wheel wheel_side="right" offset_y="${-wheel_track / 2}"/>
   <!-- Caster Wheel Pairs (Front & Back) -->
-  <caster_pair location="front" offset_x="0.650"  offset_y="0.400" mass="5.2"/>
-  <caster_pair location="back"  offset_x="-0.650" offset_y="0.400" mass="0.01"/>
+  <caster_pair location="front" offset_x="${caster_offset_x}"  offset_y="${caster_offset_y}" mass="${caster_mass}"/>
+  <caster_pair location="back"  offset_x="${-caster_offset_x}" offset_y="${caster_offset_y}" mass="${caster_mass}"/>
   <!-- 2D & 3D LiDAR Sensors (Kinematics + Simulation Stream) -->
   <lidar_sensor name="front_lidar" x="${front_lidar_x}" y="${front_lidar_y}" z="${front_lidar_z}" roll="${front_lidar_roll}" pitch="${front_lidar_pitch}" yaw="${front_lidar_yaw}" topic_name="/front_lidar/scan"/>
